Commit message: Clean stale comments from robot stack

File: ros2_ws/description/urdf/diffbot.urdf.xacro (robot description, xacro)
@@ -1,11 +1,8 @@
 <?xml version="1.0"?>
-<!-- Basic differential drive mobile base -->
 <robot xmlns:xacro="http://www.ros.org/wiki/xacro" name="diffdrive_robot">
   <xacro:arg name="prefix" default="" />
   <xacro:arg name="use_mock_hardware" default="false" />
   <xacro:include filename="$(find diffbot)/urdf/diffbot_description.urdf.xacro" />
-  <!-- Import Rviz colors -->
   <xacro:include filename="$(find diffbot)/urdf/diffbot.materials.xacro" />
-  <!-- Import diffbot ros2_control description -->
   <xacro:include filename="$(find diffbot)/ros2_control/diffbot.ros2_control.xacro" />
   <xacro:diffbot prefix="$(arg prefix)" />

File: ros2_ws/description/urdf/diffbot_description.urdf.xacro (robot description, xacro)
@@ -2,7 +2,6 @@
 <robot xmlns:xacro="http://www.ros.org/wiki/xacro">
   <xacro:macro name="diffbot" params="prefix">
-    <!-- Constants for robot dimensions -->
     <xacro:property name="PI" value="3.1415926535897931"/>
-    <xacro:property name="base_mass" value="3.4"/> <!-- arbitrary value for base mass -->
+    <xacro:property name="base_mass" value="3.4"/>
     <xacro:property name="base_width" value="0.24"/>
     <xacro:property name="base_length" value="0.13"/>
@@ -12,8 +11,8 @@
     <xacro:property name="wheel_z_offset" value="0.1"/>
     <xacro:property name="wheel_separation" value="0.2"/>
-    <xacro:property name="wheel_mass" value="0.3"/> <!-- arbitrary value for wheel mass -->
+    <xacro:property name="wheel_mass" value="0.3"/>
     <xacro:property name="wheel_len" value="0.030"/>
     <xacro:property name="wheel_radius" value="0.036"/>
-    <xacro:property name="z_offset" value="-${base_height/2}"/> <!-- Space btw top of beam and the each joint -->
+    <xacro:property name="z_offset" value="-${base_height/2}"/>
     <link name="base_footprint">
       <visual>
@@ -25,5 +24,4 @@
       </visual>
     </link>
-    <!-- Base Link -->
     <link name="${prefix}base_link">
       <visual>
@@ -43,6 +41,4 @@
       </inertial>
       <visual>
-        <!--        TODO: was: -->
-<!--        <origin xyz="0 0 ${base_height/2}" rpy="0 0 0"/>-->
         <origin xyz="0 0 0" rpy="0 0 0"/>
         <geometry>
@@ -71,5 +67,4 @@
       <limit effort="100" velocity="1.0"/>
     </joint>
-    <!-- left wheel Link -->
     <link name="${prefix}left_wheel">
       <collision>
@@ -103,5 +98,4 @@
       <limit effort="100" velocity="1.0"/>
     </joint>
-    <!-- right wheel Link -->
     <link name="${prefix}right_wheel">
       <collision>
@@ -127,7 +121,4 @@
       </inertial>
     </link>
-    <!-- ============================= -->
-    <!-- Laser -->
-    <!-- ============================= -->
     <link name="scan">
       <visual>
@@ -144,7 +135,4 @@
       <origin xyz="-0.0725 0 0.11" rpy="0 0 0"/>
     </joint>
-    <!-- ============================= -->
-    <!-- Camera -->
-    <!-- ============================= -->
     <link name="camera_link">
       <visual>
@@ -159,10 +147,6 @@
       <parent link="base_link"/>
       <child link="camera_link"/>
-      <!-- Approximate front-top mount for the RealSense body. -->
       <origin xyz="0.105 0 0.085" rpy="0 0 0"/>
     </joint>
-    <!-- ============================= -->
-    <!-- IMU (future) -->
-    <!-- ============================= -->
     <link name="imu_link">
       <visual>
@@ -177,5 +161,4 @@
       <parent link="base_link"/>
       <child link="imu_link"/>
-      <!--  TODO: validate     -->
       <origin xyz="0 0 -0.005" rpy="0 0 -${PI/2}"/>
     </joint>
